Commit message: Added IK solver ROS class and State Machine

File: garbage_quick_sort_robot_moveit_config/config/gazebo_garbage_quick_sort_robot.urdf (robot description, URDF)
Before this commit: robot garbage_quick_sort_robot, 5 links, 4 joints
Joints:
- joint joint_2: axis 0 -1 0 -> 0 1 0
- joint joint_3: axis 0 -1 0 -> 0 1 0
- joint joint_4: axis 0 -1 0 -> 0 1 0
