Commit message: changes before starting software test

File: garbage_quick_sort_robot/urdf/garbage_quick_sort_robot.urdf (robot description, URDF)
Before this commit: robot garbage_quick_sort_robot, 5 links, 4 joints
Links:
- link base_link: mass 0.015708 -> 0.015707963267949
- link link_1: mass 0.098659 -> 0.0985454479856908
- link link_2: mass 0.060349 -> 0.0483487129594158
- link link_3: mass 0.060536 -> 0.0605358880934335
- link link_4: mass 0.028481 -> 0.0426411677610806
Joints:
- joint joint_2: origin xyz=0 0 0.13138 rpy=0 0 0 -> xyz=0 0 0.131 rpy=0 0 0
- joint joint_3: origin xyz=0.236 0 0 rpy=0 0 0 -> xyz=0.186 0 0 rpy=0 0 0

File: garbage_quick_sort_robot_moveit_config/config/gazebo_garbage_quick_sort_robot.urdf (robot description, URDF)
Before this commit: robot garbage_quick_sort_robot, 5 links, 4 joints
Links:
- link base_link: mass 0.015708 -> 0.015707963267949
- link link_1: mass 0.098659 -> 0.0985454479856908
- link link_2: mass 0.060349 -> 0.0483487129594158
- link link_3: mass 0.060536 -> 0.0605358880934335
- link link_4: mass 0.028481 -> 0.0426411677610806
Joints:
- joint joint_2: axis 0 1 0 -> 0 -1 0; origin xyz=0 0 0.13138 rpy=0 0 0 -> xyz=0 0 0.131 rpy=0 0 0
- joint joint_3: axis 0 1 0 -> 0 -1 0; origin xyz=0.236 0 0 rpy=0 0 0 -> xyz=0.186 0 0 rpy=0 0 0
- joint joint_4: axis 0 1 0 -> 0 -1 0
